File: KiCad Files/LoChord/LoChord.kicad_pcb (KiCad board)
At the start: 2 copper layers, 98.5 x 96.2 mm, 25 parts, among them J1 Conn_01x07_Pin, SW1 RotaryEncoder_Switch_MP, U1 Waveshare ESP32-S3-ZERO

Commit message: PCB Done
Parts:
- removed the REF** at (139.0, 41.0)
Connections:
- D11 pad 2: Net-(D10-DOUT) -> Net-(D11-DIN)
- D11 pad 4: Net-(D11-DOUT) -> Net-(D10-DIN)
- D12 pad 2: Net-(D11-DOUT) -> unconnected-(D12-DIN-Pad2)
- D12 pad 4: unconnected-(D12-DOUT-Pad4) -> Net-(D11-DIN)
- D7 pad 2: /LED -> Net-(D7-DIN)
- D7 pad 4: Net-(D7-DOUT) -> /LED
- D8 pad 2: Net-(D7-DOUT) -> Net-(D8-DIN)
- D8 pad 4: Net-(D8-DOUT) -> Net-(D7-DIN)
- D9 pad 2: Net-(D8-DOUT) -> Net-(D10-DOUT)
- D9 pad 4: Net-(D10-DIN) -> Net-(D8-DIN)
- U1 pad 1: /COL1 -> /COL3
- U1 pad 10: /T3 -> /T4
- U1 pad 11: /T2 -> /T3
- U1 pad 12: /T1 -> /T2
- U1 pad 3: /COL3 -> /COL1
- U1 pad 6: /T7 -> /T1
- U1 pad 7: /T6 -> /T7
- U1 pad 8: /T5 -> /T6
- U1 pad 9: /T4 -> /T5
- U1 pad RX: /ROW1 -> /ROW2
- U1 pad TX: /ROW2 -> /ROW1
Routing:
- net +5V: track 0.00 -> 127.3 mm, vias 0 -> 4
- net /COL1: track 0.00 -> 121.4 mm
- net /COL2: track 0.00 -> 100.6 mm
- net /LED: track 0.00 -> 98.2 mm, vias 0 -> 1
- net /T2: track 0.00 -> 92.4 mm, vias 0 -> 2
- net /T1: track 0.00 -> 89.3 mm, vias 0 -> 1
- net /T3: track 0.00 -> 86.5 mm, vias 0 -> 1
- net /ROW2: track 0.00 -> 85.4 mm
- net /ROW1: track 0.00 -> 81.6 mm
- net /COL3: track 0.00 -> 78.8 mm, vias 0 -> 2
- net /T5: track 0.00 -> 71.5 mm, vias 0 -> 1
- net Net-(D10-DOUT): track 0.00 -> 63.9 mm, vias 0 -> 2
- net /T7: track 0.00 -> 60.2 mm, vias 0 -> 1
- net /T4: track 0.00 -> 58.2 mm
- net /T6: track 0.00 -> 32.7 mm, vias 0 -> 2
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- added copper zone on B.Cu, net GND
- added copper zone on F.Cu, net GND
Other:
- outline, holes or cut-outs redrawn
- board text added: "By Aahan P"
- board text added: "LoChord"
- board text added: "Made with love on Earth by a Human."
- board text added: "v1"
