File: KiCad Files/LoChord/LoChord.kicad_sch (KiCad schematic)
At the start: 21 parts, among them J1 Conn_01x07_Pin, SW1 RotaryEncoder_Switch_MP, U1 Waveshare ESP32-S3-ZERO

Commit message: PCB Done
Connections:
- net COL1: now also U1.3 (GP3); no longer U1.1 (GP1)
- net COL3: now also U1.1 (GP1); no longer U1.3 (GP3)
- net LED: now also D7.4 (DOUT); no longer D7.2 (DIN)
- net ROW1: now also U1.TX; no longer U1.RX
- net ROW2: now also U1.RX; no longer U1.TX
- net T1: now also U1.6 (GP6); no longer U1.12 (GP12)
- net T2: now also U1.12 (GP12); no longer U1.11 (GP11)
- net T3: now also U1.11 (GP11); no longer U1.10 (GP10)
- net T4: now also U1.10 (GP10); no longer U1.9 (GP9)
- net T5: now also U1.9 (GP9); no longer U1.8 (GP8)
- net T6: now also U1.8 (GP8); no longer U1.7 (GP7)
- net T7: now also U1.7 (GP7); no longer U1.6 (GP6)
- net at D11.2 (DIN): now also D12.4 (DOUT); no longer D10.4 (DOUT)
- net at D11.4 (DOUT): now also D10.2 (DIN); no longer D12.2 (DIN)
- net at D8.2 (DIN): now also D9.4 (DOUT); no longer D7.4 (DOUT)
- net at D8.4 (DOUT): now also D7.2 (DIN); no longer D9.2 (DIN)
- new net: D10.4 (DOUT), D9.2 (DIN)
